File: main.brd (EAGLE design)
At the start: 25.1 x 25 mm, 31 parts, among them IC1 ATTINY13A-SSH, T1A 2N4401, T1B NPN, T2A 2N4401, T2B NPN

Commit message: pcb adjustments
Parts:
- removed C1A: 100nF, capacitor-wima:C2.5-2
- removed C1B: 100nF, eagle-ltspice:C0805
- added R3, R7: 510, resistor:M0805
- added R8: 10k, resistor:M0805
- added SENSOR-: (no value), wirepad:1,6/0,8
- moved R2 10.1 mm to (21.8, 20.6)
- moved R4 5.95 mm to (9.14, 5.03)
- moved PAD1 4.18 mm to (15.4, 3.40)
- moved PAD2 4.04 mm to (11.9, 3.40)
- moved LED1 3.69 mm to (13.5, 5.89)
- moved R1 2.39 mm to (22.7, 17.5), turned to 270 degrees
- renumbered C1 to C2, PAD12 to BAT+
Connections:
- new net N$3: LED1.A, PAD1.1, R3.2, R4.2
- new net N$7: R7.1, R8.2, SENSOR-.1
- net GND: now also R8.1; no longer C1A.2, C1B.1
- net LED: now also R3.1; no longer LED1.A, PAD1.1, R4.2
- net SENSOR: now also R7.2
- net VCC: no longer C1A.1, C1B.2
Routing:
- net LED: track 33.1 -> 6.51 mm
- net N$3: track 0.00 -> 23.7 mm
- net N$7: track 0.00 -> 11.5 mm, vias 0 -> 1
- net SENSOR: track 2.48 -> 10.8 mm
- net PUMP: track 19.3 -> 24.6 mm
- net N$1: track 14.5 -> 17.2 mm
- net VCC: track 5.37 -> 2.88 mm
Other:
- board size 25.1 x 25 mm -> 25.1 x 24.8 mm

Commit message: a few more corrections
Parts:
- added C1: 100nF, rcl:C0805
Connections:
- net GND: now also C1.2
- net VCC: now also C1.1
Routing:
- net VCC: track 2.88 -> 5.03 mm
Changed lines of the file:
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@@
 </element>
 <element name="PUMP+" library="wirepad" library_urn="urn:adsk.eagle:library:412" package="2,15/1,0" package3d_urn="urn:adsk.eagle:package:30831/1" value="" x="22.86" y="14.0208" smashed="yes" rot="R90">
-<attribute name="NAME" x="25.1968" y="9.7536" size="1.27" layer="25" ratio="10" rot="R90"/>
+<attribute name="NAME" x="25.3492" y="9.7536" size="1.27" layer="25" ratio="10" rot="R90"/>
 <attribute name="VALUE" x="22.26" y="14.0208" size="0.0254" layer="27" rot="R90"/>
 </element>
@@
 </element>
 <element name="R1" library="resistor" library_urn="urn:adsk.eagle:library:348" package="M0805" package3d_urn="urn:adsk.eagle:package:23556/1" value="510" x="22.7076" y="17.526" smashed="yes" rot="R270">
-<attribute name="NAME" x="20.1676" y="18.1864" size="1.27" layer="25" rot="R270"/>
+<attribute name="NAME" x="20.4724" y="19.4056" size="1.27" layer="25" rot="R270"/>
 <attribute name="VALUE" x="20.1676" y="18.796" size="1.27" layer="27" rot="R270"/>
 </element>
@@
 </element>
 <element name="T2A" library="transistor" library_urn="urn:adsk.eagle:library:402" package="TO92" package3d_urn="urn:adsk.eagle:package:29893/2" value="2N4401" x="22.86" y="10.2108" smashed="yes" rot="R90">
-<attribute name="NAME" x="21.3106" y="11.0998" size="1.27" layer="25" ratio="10" rot="R90"/>
+<attribute name="NAME" x="21.3106" y="10.795" size="1.27" layer="25" ratio="10" rot="R90"/>
 <attribute name="VALUE" x="24.13" y="13.3858" size="1.27" layer="27" ratio="10" rot="R90"/>
 </element>
@@
 <attribute name="NAME" x="9.2964" y="6.8072" size="1.27" layer="25" ratio="10"/>
 <attribute name="VALUE" x="11.7348" y="9.4392" size="0.0254" layer="27"/>
+</element>
+<element name="C1" library="rcl" library_urn="urn:adsk.eagle:library:334" package="C0805" package3d_urn="urn:adsk.eagle:package:23617/2" value="100nF" x="20.2692" y="15.5448" smashed="yes" rot="R270">
+<attribute name="NAME" x="18.1864" y="17.1196" size="1.27" layer="25"/>
+<attribute name="SPICEPREFIX" value="C" x="20.2692" y="15.5448" size="1.778" layer="27" rot="R270" display="off"/>
+<attribute name="VALUE" x="17.7292" y="16.8148" size="1.27" layer="27" rot="R270"/>
 </element>
 </elements>
@@
 <contactref element="PAD2" pad="1"/>
 <contactref element="R8" pad="1"/>
+<contactref element="C1" pad="2"/>
 </signal>
 <signal name="N$1">
@@
 <wire x1="19.1262" y1="20.574" x2="18.1356" y2="19.5834" width="0.1524" layer="1"/>
 <wire x1="18.1356" y1="19.5834" x2="16.3068" y2="19.5834" width="0.1524" layer="1"/>
-<wire x1="22.7076" y1="18.476" x2="21.3004" y2="18.476" width="0.1524" layer="1"/>
-<wire x1="20.8432" y1="18.9332" x2="20.8432" y2="20.574" width="0.1524" layer="1"/>
-<wire x1="21.3004" y1="18.476" x2="20.8432" y2="18.9332" width="0.1524" layer="1"/>
+<wire x1="22.7076" y1="18.476" x2="21.6052" y2="18.476" width="0.1524" layer="1"/>
+<wire x1="20.8432" y1="19.238" x2="20.8432" y2="20.574" width="0.1524" layer="1"/>
+<wire x1="21.6052" y1="18.476" x2="20.8432" y2="19.238" width="0.1524" layer="1"/>
 </signal>
 <signal name="N$2">
@@
 <wire x1="19.812" y1="7.808" x2="18.288" y2="6.284" width="0.1524" layer="1"/>
 <wire x1="18.288" y1="5.8268" x2="18.288" y2="6.284" width="0.1524" layer="1"/>
-<wire x1="19.812" y1="12.954" x2="18.774228125" y2="13.991771875" width="0.1524" layer="1"/>
-<wire x1="18.774228125" y1="13.991771875" x2="18.1356" y2="14.0208" width="0.1524" layer="1"/>
-<wire x1="19.812" y1="7.808" x2="19.812" y2="12.954" width="0.1524" layer="1"/>
+<wire x1="19.812" y1="12.3444" x2="18.1356" y2="14.0208" width="0.1524" layer="1"/>
+<wire x1="19.812" y1="7.808" x2="19.812" y2="12.3444" width="0.1524" layer="1"/>
 </signal>
 <signal name="VCC">
@@
 <wire x1="15.9766" y1="14.7066" x2="16.383" y2="14.7066" width="0.1524" layer="1"/>
 <wire x1="16.383" y1="14.7066" x2="18.1356" y2="16.4592" width="0.1524" layer="1"/>
+<contactref element="C1" pad="1"/>
+<wire x1="20.2692" y1="16.4948" x2="20.2336" y2="16.4592" width="0.1524" layer="1"/>
+<wire x1="20.2336" y1="16.4592" x2="18.1356" y2="16.4592" width="0.1524" layer="1"/>
 </signal>
 <signal name="SENSOR">
@@
 <wire x1="15.9766" y1="10.8966" x2="13.1826" y2="10.8966" width="0.1524" layer="1"/>
 <wire x1="13.1826" y1="10.8966" x2="12.8016" y2="11.2776" width="0.1524" layer="1"/>
-<wire x1="12.6492" y1="18.1356" x2="18.90370625" y2="18.1356" width="0.1524" layer="1"/>
+<wire x1="12.6492" y1="18.1356" x2="20.88490625" y2="18.1356" width="0.1524" layer="1"/>
 <wire x1="11.8872" y1="17.3736" x2="12.6492" y2="18.1356" width="0.1524" layer="1"/>
-<wire x1="18.90370625" y1="18.1356" x2="20.46330625" y2="16.576" width="0.1524" layer="1"/>
-<wire x1="20.46330625" y1="16.576" x2="22.7076" y2="16.576" width="0.1524" layer="1"/>
+<wire x1="22.7076" y1="16.576" x2="22.44450625" y2="16.576" width="0.1524" layer="1"/>
+<wire x1="22.44450625" y1="16.576" x2="20.88490625" y2="18.1356" width="0.1524" layer="1"/>
 <wire x1="12.8016" y1="11.2776" x2="12.8016" y2="15.24" width="0.1524" layer="1"/>
 <wire x1="12.8016" y1="15.24" x2="11.8872" y2="16.1544" width="0.1524" layer="1"/>

Commit message: optimized pcb and code
Parts:
- removed R8: 10k, resistor:M0805
- R7: value 510 -> 10k
- moved REG1 22.1 mm to (22.7, 6.25), turned to 90 degrees
- moved T2A 20.9 mm to (3.51, 18.1), turned to 270 degrees
- moved T2B 20.3 mm to (8.23, 20.7), turned to 270 degrees
- moved R1 9.72 mm to (13.3, 19.8), turned to 180 degrees
- moved R2 8.64 mm to (13.3, 21.9), turned to 0 degrees
- moved SENSOR- 8.06 mm to (13.9, 16.6)
- moved T1B 7.77 mm to (17.5, 20.9), turned to 90 degrees
- moved T1A 7.23 mm to (22.7, 18.1), turned to 90 degrees
- moved R4 6.14 mm to (4.72, 9.30), turned to 180 degrees
- moved C1 5.17 mm to (21.5, 10.5)
- moved R6 4.73 mm to (8.99, 5.03), turned to 270 degrees
- moved C2 4.13 mm to (4.57, 4.88), turned to 180 degrees
- moved PAD1 3.20 mm to (12.2, 3.40)
- moved PAD2 3.05 mm to (15.0, 3.40)
- moved R3 3.03 mm to (4.72, 11.4), turned to 180 degrees
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Connections:
- removed net N$7: R7.1, R8.2, SENSOR-.1
- net GND: now also R7.1; no longer R8.1
- net SENSOR: now also SENSOR-.1
Routing:
- net N$6: track 26.1 -> 4.16 mm
- net N$7: track 11.5 -> 0.00 mm, vias 1 -> 0
- net N$2: track 21.4 -> 31.9 mm
- net SOLAR_PANEL+: track 10.8 -> 21.2 mm
- net PUMP: track 24.6 -> 15.1 mm
- net N$4: track 30.3 -> 38.8 mm
- net N$3: track 23.7 -> 15.2 mm
- net GND: track 0.00 -> 8.12 mm
- net N$5: track 36.4 -> 29.1 mm
- net SENSOR: track 10.8 -> 18.1 mm
- net N$1: track 17.0 -> 10.4 mm
- net VCC: track 5.03 -> 10.8 mm
- net LED: track 6.51 -> 9.99 mm
Other:
- board text added: "Rev 0.2"
- board text removed: "Rev 0.1"

Commit message: Rev 0.3
Parts:
- added SENSOR+: (no value), wirepad:1,6/0,8
- moved SENSOR- 2.41 mm to (11.6, 17.4)
Connections:
- removed net SENSOR: IC1.6, PAD6.1, R7.2, SENSOR-.1
- removed net UART_RX: IC1.3, PAD8.1
- new net SENSOR+: IC1.6, PAD6.1, SENSOR+.1
- new net SENSOR-: IC1.3, PAD8.1, R7.1, SENSOR-.1
- net GND: now also R7.2; no longer R7.1
Routing:
- net SENSOR: track 18.1 -> 0.00 mm
- net SENSOR-: track 0.00 -> 13.6 mm
- net SENSOR+: track 0.00 -> 9.77 mm
- net N$5: track 29.1 -> 31.7 mm
- net UART_RX: track 2.46 -> 0.00 mm
- net PUMP: track 15.1 -> 14.5 mm
Other:
- board text added: "Rev 0.3"
- board text removed: "Rev 0.2"
Changed lines of the file:
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@@
 <text x="2.5908" y="20.8788" size="1.27" layer="25">BAT-</text>
 <text x="19.6596" y="20.7264" size="1.27" layer="25">BAT+</text>
-<text x="0.9144" y="24.2316" size="1.27" layer="25" rot="R270">Rev 0.2</text>
+<text x="0.9144" y="24.2316" size="1.27" layer="25" rot="R270">Rev 0.3</text>
 </plain>
 <attributes>
@@
 <attribute name="VALUE" x="12.2936" y="5.9944" size="1.27" layer="27"/>
 </element>
-<element name="SENSOR-" library="wirepad" library_urn="urn:adsk.eagle:library:412" package="1,6/0,8" package3d_urn="urn:adsk.eagle:package:30830/1" value="" x="13.8684" y="16.6116" smashed="yes">
-<attribute name="NAME" x="9.7536" y="17.4752" size="1.27" layer="25" ratio="10"/>
-<attribute name="VALUE" x="13.8684" y="17.2116" size="0.0254" layer="27"/>
+<element name="SENSOR+" library="wirepad" library_urn="urn:adsk.eagle:library:412" package="1,6/0,8" package3d_urn="urn:adsk.eagle:package:30830/1" value="" x="15.5448" y="17.3736" smashed="yes">
+<attribute name="NAME" x="11.43" y="18.2372" size="1.27" layer="25" ratio="10"/>
+<attribute name="VALUE" x="15.5448" y="17.9736" size="0.0254" layer="27"/>
 </element>
 <element name="C1" library="rcl" library_urn="urn:adsk.eagle:library:334" package="C0805" package3d_urn="urn:adsk.eagle:package:23617/2" value="100nF" x="21.4884" y="10.5156" smashed="yes" rot="R270">
@@
 <attribute name="SPICEPREFIX" value="C" x="21.4884" y="10.5156" size="1.778" layer="27" rot="R270" display="off"/>
 <attribute name="VALUE" x="18.9484" y="11.7856" size="1.27" layer="27" rot="R270"/>
+</element>
+<element name="SENSOR-" library="wirepad" library_urn="urn:adsk.eagle:library:412" package="1,6/0,8" package3d_urn="urn:adsk.eagle:package:30830/1" value="" x="11.5824" y="17.3736" smashed="yes">
+<attribute name="NAME" x="10.8204" y="18.3896" size="1.27" layer="25" ratio="10"/>
+<attribute name="VALUE" x="11.5824" y="17.9736" size="0.0254" layer="27"/>
 </element>
 </elements>
@@
 <wire x1="8.89" y1="14.0208" x2="9.4742" y2="13.4366" width="0.1524" layer="1"/>
 <wire x1="9.4742" y1="13.4366" x2="11.049" y2="13.4366" width="0.1524" layer="1"/>
-</signal>
-<signal name="UART_RX">
-<contactref element="IC1" pad="3"/>
-<contactref element="PAD8" pad="1"/>
-<wire x1="8.89" y1="11.43" x2="9.6266" y2="12.1666" width="0.1524" layer="1"/>
-<wire x1="9.6266" y1="12.1666" x2="11.049" y2="12.1666" width="0.1524" layer="1"/>
 </signal>
 <signal name="GND">
@@
 <contactref element="LED1" pad="C"/>
 <contactref element="PAD2" pad="1"/>
-<contactref element="R7" pad="1"/>
 <contactref element="C1" pad="2"/>
 <wire x1="5.7404" y1="8.8392" x2="3.302" y2="6.4008" width="0.3048" layer="16"/>
 <wire x1="3.302" y1="4.8768" x2="3.302" y2="6.4008" width="0.3048" layer="16"/>
 <wire x1="5.7404" y1="8.8392" x2="8.89" y2="8.8392" width="0.3048" layer="16"/>
+<contactref element="R7" pad="2"/>
 </signal>
 <signal name="N$1">
@@
 <wire x1="20.6222" y1="18.1356" x2="18.829" y2="19.9288" width="0.1524" layer="1"/>
 <wire x1="14.2088" y1="21.9456" x2="14.2088" y2="19.812" width="0.1524" layer="1"/>
-<wire x1="14.2088" y1="19.812" x2="15.2756" y2="18.7452" width="0.1524" layer="1"/>
-<wire x1="15.2756" y1="18.7452" x2="17.6454" y2="18.7452" width="0.1524" layer="1"/>
-<wire x1="17.6454" y1="18.7452" x2="18.829" y2="19.9288" width="0.1524" layer="1"/>
+<wire x1="14.2088" y1="19.812" x2="15.1232" y2="18.8976" width="0.1524" layer="1"/>
+<wire x1="15.1232" y1="18.8976" x2="17.7978" y2="18.8976" width="0.1524" layer="1"/>
+<wire x1="17.7978" y1="18.8976" x2="18.829" y2="19.9288" width="0.1524" layer="1"/>
 </signal>
 <signal name="N$2">
@@
 <wire x1="15.9766" y1="15.621" x2="15.9766" y2="14.7066" width="0.1524" layer="1"/>
 </signal>
-<signal name="SENSOR">
+<signal name="SENSOR+">
 <contactref element="IC1" pad="6"/>
 <contactref element="PAD6" pad="1"/>
 <wire x1="18.1356" y1="11.43" x2="17.4498" y2="12.1666" width="0.1524" layer="1"/>
 <wire x1="17.4498" y1="12.1666" x2="15.9766" y2="12.1666" width="0.1524" layer="1"/>
-<wire x1="18.7452" y1="7.4676" x2="17.1044" y2="7.4676" width="0.1524" layer="1"/>
-<wire x1="18.7452" y1="7.4676" x2="19.3548" y2="8.0772" width="0.1524" layer="1"/>
-<wire x1="19.3548" y1="8.0772" x2="19.3548" y2="10.2108" width="0.1524" layer="1"/>
-<wire x1="19.3548" y1="10.2108" x2="18.1356" y2="11.43" width="0.1524" layer="1"/>
-<contactref element="R7" pad="2"/>
-<contactref element="SENSOR-" pad="1"/>
-<wire x1="13.8684" y1="16.6116" x2="13.8684" y2="12.6492" width="0.1524" layer="1"/>
-<wire x1="14.351" y1="12.1666" x2="15.9766" y2="12.1666" width="0.1524" layer="1"/>
-<wire x1="13.8684" y1="12.6492" x2="14.351" y2="12.1666" width="0.1524" layer="1"/>
-<wire x1="17.1044" y1="7.4676" x2="16.0376" y2="8.5344" width="0.1524" layer="1"/>
-<wire x1="16.0376" y1="8.5344" x2="14.5136" y2="8.5344" width="0.1524" layer="1"/>
+<wire x1="15.9766" y1="12.1666" x2="14.4526" y2="12.1666" width="0.1524" layer="1"/>
+<wire x1="14.4526" y1="12.1666" x2="14.3256" y2="12.2936" width="0.1524" layer="1"/>
+<contactref element="SENSOR+" pad="1"/>
+<wire x1="15.5448" y1="17.3736" x2="14.3256" y2="16.1544" width="0.1524" layer="1"/>
+<wire x1="14.3256" y1="16.1544" x2="14.3256" y2="12.2936" width="0.1524" layer="1"/>
 </signal>
 <signal name="PUMP">
@@
 <wire x1="15.9766" y1="10.8966" x2="17.9832" y2="8.89" width="0.1524" layer="1"/>
 <wire x1="17.9832" y1="8.89" x2="18.1356" y2="8.8392" width="0.1524" layer="1"/>
-<wire x1="15.9766" y1="10.8966" x2="13.335" y2="10.8966" width="0.1524" layer="1"/>
-<wire x1="13.335" y1="10.8966" x2="12.8016" y2="11.43" width="0.1524" layer="1"/>
-<wire x1="12.3088" y1="19.812" x2="12.192" y2="19.6952" width="0.1524" layer="1"/>
-<wire x1="12.192" y1="19.6952" x2="12.192" y2="15.8496" width="0.1524" layer="1"/>
-<wire x1="12.8016" y1="11.43" x2="12.8016" y2="15.24" width="0.1524" layer="1"/>
-<wire x1="12.8016" y1="15.24" x2="12.192" y2="15.8496" width="0.1524" layer="1"/>
+<wire x1="15.9766" y1="10.8966" x2="14.097" y2="10.8966" width="0.1524" layer="1"/>
+<wire x1="14.097" y1="10.8966" x2="13.5636" y2="11.43" width="0.1524" layer="1"/>
+<wire x1="13.5636" y1="18.2524" x2="12.3088" y2="19.5072" width="0.1524" layer="1"/>
+<wire x1="12.3088" y1="19.812" x2="12.3088" y2="19.5072" width="0.1524" layer="1"/>
+<wire x1="13.5636" y1="18.2524" x2="13.5636" y2="11.43" width="0.1524" layer="1"/>
 </signal>
 <signal name="N$4">
@@
 <wire x1="6.9266" y1="19.7764" x2="3.876" y2="19.7764" width="0.1524" layer="1"/>
 <wire x1="3.876" y1="19.7764" x2="3.5052" y2="19.4056" width="0.1524" layer="1"/>
-<wire x1="8.0772" y1="19.812" x2="3.9116" y2="19.812" width="0.3048" layer="16"/>
+<wire x1="12.3444" y1="19.812" x2="3.9116" y2="19.812" width="0.3048" layer="16"/>
 <wire x1="3.5052" y1="19.4056" x2="3.9116" y2="19.812" width="0.3048" layer="16"/>
-<wire x1="16.1544" y1="11.7348" x2="16.1544" y2="7.62" width="0.3048" layer="16"/>
-<wire x1="16.1544" y1="7.62" x2="17.526" y2="6.2484" width="0.3048" layer="16"/>
-<wire x1="17.526" y1="6.2484" x2="20.8026" y2="6.2484" width="0.3048" layer="16"/>
-<wire x1="8.0772" y1="19.812" x2="16.1544" y2="11.7348" width="0.3048" layer="16"/>
+<wire x1="13.5636" y1="18.5928" x2="13.5636" y2="9.906" width="0.3048" layer="16"/>
+<wire x1="13.5636" y1="9.906" x2="17.2212" y2="6.2484" width="0.3048" layer="16"/>
+<wire x1="17.2212" y1="6.2484" x2="20.8026" y2="6.2484" width="0.3048" layer="16"/>
+<wire x1="12.3444" y1="19.812" x2="13.5636" y2="18.5928" width="0.3048" layer="16"/>
 </signal>
 <signal name="SOLAR_PANEL+">
@@
 <wire x1="7.62" y1="16.4592" x2="8.89" y2="16.4592" width="0.1524" layer="1"/>
 </signal>
-<signal name="SENSOR+">
+<signal name="SENSOR-">
+<contactref element="IC1" pad="3"/>
+<contactref element="PAD8" pad="1"/>
+<wire x1="8.89" y1="11.43" x2="9.6266" y2="12.1666" width="0.1524" layer="1"/>
+<wire x1="9.6266" y1="12.1666" x2="11.049" y2="12.1666" width="0.1524" layer="1"/>
+<contactref element="R7" pad="1"/>
+<contactref element="SENSOR-" pad="1"/>
+<wire x1="11.5824" y1="17.3736" x2="12.8016" y2="16.1544" width="0.1524" layer="1"/>
+<wire x1="12.8016" y1="16.1544" x2="12.8016" y2="12.4968" width="0.1524" layer="1"/>
+<wire x1="12.8016" y1="12.4968" x2="12.4968" y2="12.192" width="0.1524" layer="1"/>
+<wire x1="12.6136" y1="8.5344" x2="12.8016" y2="8.7224" width="0.1524" layer="1"/>
+<wire x1="12.8016" y1="8.7224" x2="12.8016" y2="11.8872" width="0.1524" layer="1"/>
+<wire x1="12.8016" y1="11.8872" x2="12.4968" y2="12.192" width="0.1524" layer="1"/>
+<wire x1="12.4968" y1="12.192" x2="12.4714" y2="12.1666" width="0.1524" layer="1"/>
+<wire x1="12.4714" y1="12.1666" x2="11.049" y2="12.1666" width="0.1524" layer="1"/>
 </signal>
 </signals>

Commit message: Rev 0.4
Parts:
- moved T2B 0.30 mm to (8.53, 20.7)
- moved C1 0.15 mm to (21.5, 10.7)
- moved T1B 0.15 mm to (17.7, 20.9)
- moved R1 0.15 mm to (13.4, 19.8)
- moved R2 0.15 mm to (13.4, 21.9)
Connections:
- removed net N$6: IN+.1, REG1.1
- net SENSOR-: now also IN+.1, REG1.1
Routing:
- net SENSOR-: track 13.6 -> 34.3 mm
- net N$6: track 4.16 -> 0.00 mm
Other:
- board text added: "Rev 0.4"
- board text removed: "Rev 0.3"

Commit message: Rev 0.5
Parts:
- removed R7: 10k, resistor:M0805
- removed REG1: 7805L, linear:TO92
- removed SENSOR+, SENSOR-: (no value), wirepad:1,6/0,8
- added REG1A: 7805L, linear:TO92
- added REG1B: LM2936MP-5.0, STM32F103RBT6:SOT230P700X180-4N
- R3: value 510 -> 120
- R4: value 10k -> 510
- R5: value 510 -> 10k
- moved PUMP+ 19.4 mm to (3.51, 14.0)
- moved PUMP- 19.2 mm to (22.9, 14.0)
- moved R4 16.1 mm to (20.3, 13.6), turned to 270 degrees
- moved C1 10.5 mm to (13.3, 17.2), turned to 180 degrees
- moved R5 9.36 mm to (8.99, 4.11)
- moved R6 5.94 mm to (13.4, 8.99), turned to 180 degrees
- moved R3 2.91 mm to (6.71, 13.6), turned to 270 degrees
- moved PAD1 2.78 mm to (11.7, 6.15)
- moved PAD2 2.75 mm to (15.1, 6.15)
- moved C2 2.14 mm to (4.42, 7.01), turned to 90 degrees
- moved LED1 2.13 mm to (13.5, 3.76)
- moved PAD3 0.30 mm to (17.8, 16.5)
- moved PAD4 0.30 mm to (17.8, 14.0)
- moved PAD5 0.30 mm to (17.8, 8.84)
- moved PAD6 0.30 mm to (17.8, 11.4)
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Connections:
- net GND: now also R5.1, R6.2; no longer R4.1, R6.1, R7.2
- net N$3: no longer R4.2
- net N$4: now also R4.2; no longer R6.2
- net N$5: now also REG1A.2, REG1B.2, REG1B.4; no longer REG1.2
- net SENSOR+: no longer SENSOR+.1
- net SENSOR-: now also R6.1, REG1A.1, REG1B.3; no longer R7.1, REG1.1, SENSOR-.1
- net SOLAR: now also R4.1; no longer R5.1
- net SOLAR_PANEL+: now also REG1A.3, REG1B.1; no longer REG1.3
Routing:
- net N$2: track 31.9 -> 12.9 mm
- net N$5: track 32.1 -> 48.3 mm
- net SOLAR_PANEL+: track 21.2 -> 37.0 mm
- net N$4: track 38.8 -> 49.1 mm
- net GND: track 8.12 -> 0.00 mm
- net SENSOR+: track 9.77 -> 2.38 mm
- net SOLAR: track 12.3 -> 4.99 mm
- net SENSOR-: track 34.3 -> 39.6 mm
- net LED: track 9.99 -> 6.55 mm
- net VCC: track 10.6 -> 7.21 mm
- net PUMP: track 14.5 -> 17.4 mm
- net N$3: track 15.2 -> 12.6 mm
Other:
- board text added: "Rev 0.5"
- board text removed: "Rev 0.4"

Commit message: code updates
Parts:
- removed R3: 120, resistor:M0805
- moved PAD10 0.91 mm to (7.98, 16.5)
- moved PAD7 0.91 mm to (7.98, 8.84)
- moved PAD8 0.91 mm to (7.98, 11.4)
- moved PAD9 0.91 mm to (7.98, 14.0)
- moved PAD3 0.46 mm to (18.3, 16.5)
- moved PAD4 0.46 mm to (18.3, 14.0)
- moved PAD5 0.46 mm to (18.3, 8.84)
- moved PAD6 0.46 mm to (18.3, 11.4)
- moved C1 0.15 mm to (13.1, 17.2)
- moved IC1 0.15 mm to (13.2, 12.8)
- moved R1 0.15 mm to (13.1, 19.8)
- moved R2 0.15 mm to (13.1, 21.9)
- moved R4 0.15 mm to (20.4, 13.6)
- moved R6 0.15 mm to (13.3, 8.99)
Connections:
- removed net N$3: LED1.A, PAD1.1, R3.2
- net LED: now also LED1.A, PAD1.1; no longer R3.1
Routing:
- net LED: track 6.55 -> 21.6 mm
- net N$3: track 12.6 -> 0.00 mm
- net SENSOR-: track 39.6 -> 41.3 mm
- net VCC: track 7.21 -> 8.34 mm
- net UART_TX: track 2.25 -> 3.01 mm
- net SENSOR+: track 2.38 -> 2.99 mm

Commit message: rev 0.6
Parts:
- removed IN-: 5V, wirepad:1,6/0,9
- removed PAD2: (no value), wirepad:1,6/0,8
- removed T2A: 2N4401, transistor:TO92
- removed T2B: NPN, semicon-smd-ipc:SOT23W
- added C3, C4: 10uF, rcl:C3216
- added IC2: TP4056-42-ESOP8, 1EDI60I12AF:SOIC127P600X175-9N
- added LED2: (no value), led:SML0805
- added R3: 10k, resistor:M0805
- added R7: 510, resistor:M0805
- added R8: 10k, rcl:R0603
- added R9: 1.2k, rcl:R0603
- R4: value 510 -> R400; device resistor:M0805 -> resistor:M1206
- moved LED1 19.2 mm to (13.2, 23.0)
- moved PAD1 17.2 mm to (8.38, 23.1)
- moved R5 15.1 mm to (22.9, 10.1)
- moved REG1A 11.3 mm to (13.1, 4.27)
- moved R4 9.89 mm to (16.3, 4.57), flipped to the bottom, turned to 90 degrees
- moved T1A 9.63 mm to (13.1, 18.9), turned to 0 degrees
- moved C1 9.07 mm to (22.1, 18.4), turned to 90 degrees
- moved R2 6.85 mm to (6.71, 19.5), turned to 90 degrees
- moved R1 3.82 mm to (9.30, 19.5), turned to 270 degrees
- moved C2 3.23 mm to (5.49, 3.96), turned to 270 degrees
- moved T1B 1.23 mm to (18.3, 19.7), turned to 270 degrees
- moved R6 1.23 mm to (13.1, 7.77), turned to 0 degrees
- moved PUMP+ 0.34 mm to (3.81, 14.2)
- moved PUMP- 0.15 mm to (22.9, 14.2)
Connections:
- new net N$11: IC2.2, R9.1
- new net N$3: IN+.1, R3.2, REG1A.1, REG1B.3
- new net N$6: LED1.A, PAD1.1, R7.2
- new net N$7: BAT+.1, C4.1, IC2.5
- new net N$8: IC2.7, R8.2
- new net N$9: LED2.C, R8.1
- net GND: now also C3.2, C4.2, R9.2; no longer IN-.1, PAD2.1, T2A.1, T2B.3
- net LED: now also R7.1; no longer LED1.A, PAD1.1
- net N$4: now also C3.1, IC2.4, IC2.8, LED2.A; no longer R5.2, T2A.2, T2B.1
- net N$5: now also R5.2; no longer T2A.3, T2B.2
- net SENSOR-: now also R3.1; no longer IN+.1, REG1A.1, REG1B.3
- net SOLAR: no longer R4.1
- net VCC: now also R4.1; no longer BAT+.1
Routing:
- net N$5: track 48.1 -> 17.8 mm
- net SENSOR-: track 41.3 -> 13.9 mm
- net SOLAR_PANEL+: track 37.2 -> 12.6 mm
- net N$3: track 0.00 -> 23.1 mm
- net GND: track 0.00 -> 16.2 mm
- net N$7: track 0.00 -> 15.1 mm
- net LED: track 21.6 -> 9.10 mm
- net N$2: track 12.9 -> 22.5 mm
- net N$6: track 0.00 -> 9.03 mm
- net N$8: track 0.00 -> 8.90 mm
- net N$4: track 49.4 -> 43.0 mm
- net N$11: track 0.00 -> 5.66 mm
- net PUMP: track 17.7 -> 15.2 mm
- net N$9: track 0.00 -> 2.38 mm
- net SOLAR: track 5.20 -> 2.86 mm
Other:
- board size 25.1 x 24.8 mm -> 24.8 x 24.7 mm
- board text added: "Rev 0.6"
- board text removed: "Rev 0.5"
