File: main.sch (EAGLE design)
At the start: 31 parts, among them IC1 ATTINY13A-SSH, T1A 2N4401, T1B NPN, T2A 2N4401, T2B NPN

Commit message: pcb adjustments
Parts:
- removed C1A: 100nF, capacitor-wima:C2.5/2
- removed C1B: 100nF, eagle-ltspice:C
- added R3, R7: 510, resistor:R-EU_M0805
- added R8: 10k, resistor:R-EU_M0805
- added SENSOR-: (no value), wirepad:1,6/0,8
- renumbered C1 to C2, PAD12 to BAT+
Connections:
- new net N$3: LED1.A, PAD1.P, R3.2, R4.2
- new net N$7: R7.1, R8.2, SENSOR-.P
- net GND: now also R8.1; no longer C1A.2, C1B.1
- net LED: now also R3.1; no longer LED1.A, PAD1.P, R4.2
- net SENSOR: now also R7.2
- net VCC: no longer C1A.1, C1B.2
Other:
- note added: "Battery / Input"
- note added: "Moisture Sensor"
- note removed: "Battery Charger / Input"

Commit message: a few more corrections
Parts:
- added C1: 100nF, rcl:C-EUC0805
Connections:
- net GND: now also C1.2
- net VCC: now also C1.1
Changed lines of the file:
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@@
 <part name="GND2" library="supply1" library_urn="urn:adsk.eagle:library:371" deviceset="GND" device=""/>
 <part name="P+3" library="supply1" library_urn="urn:adsk.eagle:library:371" deviceset="VCC" device=""/>
+<part name="C1" library="rcl" library_urn="urn:adsk.eagle:library:334" deviceset="C-EU" device="C0805" package3d_urn="urn:adsk.eagle:package:23617/2" value="100nF"/>
+<part name="GND6" library="supply1" library_urn="urn:adsk.eagle:library:371" deviceset="GND" device=""/>
 </parts>
 <sheets>
@@
 <attribute name="VALUE" x="114.3" y="27.94" size="1.778" layer="96" rot="R180"/>
 </instance>
+<instance part="C1" gate="G$1" x="99.06" y="48.26" smashed="yes">
+<attribute name="NAME" x="100.584" y="48.641" size="1.778" layer="95"/>
+<attribute name="VALUE" x="100.584" y="43.561" size="1.778" layer="96"/>
+</instance>
+<instance part="GND6" gate="1" x="99.06" y="40.64" smashed="yes">
+<attribute name="VALUE" x="96.52" y="38.1" size="1.778" layer="96"/>
+</instance>
 </instances>
 <busses>
@@
 <pinref part="GND2" gate="1" pin="GND"/>
 </segment>
+<segment>
+<pinref part="C1" gate="G$1" pin="2"/>
+<pinref part="GND6" gate="1" pin="GND"/>
+</segment>
 </net>
 <net name="N$1" class="0">
@@
 <segment>
 <pinref part="P+1" gate="VCC" pin="VCC"/>
-<wire x1="93.98" y1="50.8" x2="93.98" y2="40.64" width="0.1524" layer="91"/>
 <junction x="93.98" y="50.8"/>
 <pinref part="PAD3" gate="P" pin="P"/>
 <pinref part="PUMP+" gate="1" pin="P"/>
 <pinref part="IC1" gate="G$1" pin="VCC"/>
+<wire x1="93.98" y1="50.8" x2="93.98" y2="40.64" width="0.1524" layer="91"/>
 <wire x1="78.74" y1="55.88" x2="93.98" y2="55.88" width="0.1524" layer="91"/>
 <wire x1="93.98" y1="55.88" x2="99.06" y2="55.88" width="0.1524" layer="91"/>
 <wire x1="93.98" y1="50.8" x2="93.98" y2="55.88" width="0.1524" layer="91"/>
 <junction x="93.98" y="55.88"/>
-</segment>
-<segment>
+<pinref part="C1" gate="G$1" pin="1"/>
+<wire x1="93.98" y1="50.8" x2="99.06" y2="50.8" width="0.1524" layer="91"/>
+</segment>
+<segment>

Commit message: optimized pcb and code
Parts:
- removed R8: 10k, resistor:R-EU_M0805
- R7: value 510 -> 10k
Connections:
- removed net N$7: R7.1, R8.2, SENSOR-.P
- net GND: now also R7.1; no longer R8.1
- net SENSOR: now also SENSOR-.P
Other:
- moved on the sheet: C2, IN+, IN-, R5, R6, R7, REG1, T2A, T2B

Commit message: Rev 0.3
Parts:
- added SENSOR+: (no value), wirepad:1,6/0,8
Connections:
- removed net SENSOR: IC1.PB1, PAD6.P, R7.2, SENSOR-.P
- removed net UART_RX: IC1.PB4, PAD8.P
- new net SENSOR+: IC1.PB1, PAD6.P, SENSOR+.P
- new net SENSOR-: IC1.PB4, PAD8.P, R7.1, SENSOR-.P
- net GND: now also R7.2; no longer R7.1
Other:
- moved on the sheet: C1, PUMP+, PUMP-, R1, R2, R7, SENSOR-, T1A, T1B

Commit message: Rev 0.4
Connections:
- removed net N$6: IN+.P, REG1.VO
- net SENSOR-: now also IN+.P, REG1.VO
Changed lines of the file:
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@@
-</segment>
-</net>
-<net name="N$6" class="0">
-<segment>
-<pinref part="REG1" gate="A1" pin="VO"/>
-<pinref part="IN+" gate="1" pin="P"/>
-<wire x1="132.08" y1="91.44" x2="132.08" y2="81.28" width="0.1524" layer="91"/>
 </segment>
 </net>
@@
 <wire x1="132.08" y1="33.02" x2="121.92" y2="33.02" width="0.1524" layer="91"/>
 <junction x="121.92" y="33.02"/>
+<pinref part="IN+" gate="1" pin="P"/>
+<pinref part="REG1" gate="A1" pin="VO"/>
+<wire x1="132.08" y1="91.44" x2="132.08" y2="81.28" width="0.1524" layer="91"/>
+<junction x="132.08" y="81.28"/>
+<wire x1="132.08" y1="81.28" x2="139.7" y2="81.28" width="0.1524" layer="91"/>
+<wire x1="139.7" y1="81.28" x2="139.7" y2="99.06" width="0.1524" layer="91"/>
+<wire x1="139.7" y1="99.06" x2="53.34" y2="99.06" width="0.1524" layer="91"/>
+<wire x1="53.34" y1="99.06" x2="53.34" y2="58.42" width="0.1524" layer="91"/>
 </segment>
 </net>

Commit message: Rev 0.5
Parts:
- removed R7: 10k, resistor:R-EU_M0805
- removed SENSOR+, SENSOR-: (no value), wirepad:1,6/0,8
- added REG1B: LM2936MP-5.0, STM32F103RBT6:LM2936MP-5.0
- R3: value 510 -> 120
- R4: value 10k -> 510
- R5: value 510 -> 10k
- renumbered REG1 to REG1A
Connections:
- net GND: now also R5.1, R6.2; no longer R4.1, R6.1, R7.2
- net N$3: no longer R4.2
- net N$4: now also R4.2; no longer R6.2
- net N$5: now also REG1B.GND, REG1B.GND_1
- net SENSOR+: no longer SENSOR+.P
- net SENSOR-: now also R6.1, REG1B.VOUT; no longer R7.1, SENSOR-.P
- net SOLAR: now also R4.1; no longer R5.1
- net SOLAR_PANEL+: now also REG1B.VIN
Other:
- moved on the sheet: R4, R5, R6

Commit message: code updates
Parts:
- removed R3: 120, resistor:R-EU_M0805
Connections:
- removed net N$3: LED1.A, PAD1.P, R3.2
- net LED: now also LED1.A, PAD1.P; no longer R3.1
Changed lines of the file:
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@@
 <?xml version="1.0" encoding="utf-8"?>
 <!DOCTYPE eagle SYSTEM "eagle.dtd">
-<eagle version="9.3.0">
+<eagle version="9.4.2">
 <drawing>
 <settings>
@@
 <part name="GND5" library="supply1" library_urn="urn:adsk.eagle:library:371" deviceset="GND" device=""/>
 <part name="REG1A" library="linear" library_urn="urn:adsk.eagle:library:262" deviceset="78*" device="L" package3d_urn="urn:adsk.eagle:package:16416/2" technology="05"/>
-<part name="R3" library="resistor" library_urn="urn:adsk.eagle:library:348" deviceset="R-EU_" device="M0805" package3d_urn="urn:adsk.eagle:package:23556/1" value="120"/>
 <part name="R6" library="resistor" library_urn="urn:adsk.eagle:library:348" deviceset="R-EU_" device="M0805" package3d_urn="urn:adsk.eagle:package:23556/1" value="10k"/>
 <part name="C1" library="rcl" library_urn="urn:adsk.eagle:library:334" deviceset="C-EU" device="C0805" package3d_urn="urn:adsk.eagle:package:23617/2" value="100nF"/>
@@
 <attribute name="VALUE" x="114.3" y="94.615" size="1.778" layer="96"/>
 </instance>
-<instance part="R3" gate="G$1" x="27.94" y="63.5" smashed="yes" rot="R180">
-<attribute name="NAME" x="31.75" y="62.0014" size="1.778" layer="95" rot="R180"/>
-<attribute name="VALUE" x="31.75" y="66.802" size="1.778" layer="96" rot="R180"/>
-</instance>
 <instance part="R6" gate="G$1" x="116.84" y="33.02" smashed="yes" rot="R180">
 <attribute name="NAME" x="120.65" y="31.5214" size="1.778" layer="95" rot="R180"/>
@@
 </segment>
 </net>
-<net name="N$3" class="0">
-<segment>
-<pinref part="LED1" gate="G$1" pin="A"/>
-<wire x1="27.94" y1="53.34" x2="20.32" y2="53.34" width="0.1524" layer="91"/>
-<pinref part="PAD1" gate="P" pin="P"/>
-<wire x1="33.02" y1="53.34" x2="27.94" y2="53.34" width="0.1524" layer="91"/>
-<junction x="27.94" y="53.34"/>
-<wire x1="20.32" y1="63.5" x2="20.32" y2="53.34" width="0.1524" layer="91"/>
-<pinref part="R3" gate="G$1" pin="2"/>
-<wire x1="22.86" y1="63.5" x2="20.32" y2="63.5" width="0.1524" layer="91"/>
-</segment>
-</net>
 <net name="SOLAR" class="0">
 <segment>
@@
 <pinref part="PAD10" gate="P" pin="P"/>
 <pinref part="IC1" gate="G$1" pin="PB5"/>
-<pinref part="R3" gate="G$1" pin="1"/>
 <junction x="40.64" y="63.5"/>
-<wire x1="33.02" y1="63.5" x2="40.64" y2="63.5" width="0.1524" layer="91"/>
+<wire x1="27.94" y1="63.5" x2="40.64" y2="63.5" width="0.1524" layer="91"/>
 <label x="43.18" y="63.5" size="1.778" layer="95"/>
 <wire x1="40.64" y1="63.5" x2="53.34" y2="63.5" width="0.1524" layer="91"/>
-</segment>
-</net>
+<pinref part="LED1" gate="G$1" pin="A"/>
+<pinref part="PAD1" gate="P" pin="P"/>
+<wire x1="33.02" y1="53.34" x2="27.94" y2="53.34" width="0.1524" layer="91"/>
+<wire x1="27.94" y1="63.5" x2="27.94" y2="53.34" width="0.1524" layer="91"/>
+<junction x="27.94" y="53.34"/>
+</segment>
+</net>

Commit message: rev 0.6
Parts:
- removed IN-: 5V, wirepad:1,6/0,9
- removed PAD2: (no value), wirepad:1,6/0,8
- removed T2A: 2N4401, transistor:-NPN-TO92
- removed T2B: NPN, semicon-smd-ipc:NPN-TRANSISTOR_SOT23W
- added C3, C4: 10uF, rcl:C-EUC3216
- added IC2: TP4056-42-ESOP8, 1EDI60I12AF:TP4056-42-ESOP8
- added LED2: (no value), led:LEDSML0805
- added R3: 10k, resistor:R-EU_M0805
- added R7: 510, resistor:R-EU_M0805
- added R8: 10k, rcl:R-EU_R0603
- added R9: 1.2k, rcl:R-EU_R0603
- R4: value 510 -> R400; device resistor:R-EU_M0805 -> resistor:R-EU_M1206
Connections:
- new net N$11: IC2.PROG, R9.1
- new net N$3: IN+.P, R3.2, REG1A.VO, REG1B.VOUT
- new net N$6: LED1.A, PAD1.P, R7.2
- new net N$7: BAT+.P, C4.1, IC2.BAT
- new net N$8: IC2.!CHRG, R8.2
- new net N$9: LED2.C, R8.1
- net GND: now also C3.2, C4.2, R9.2; no longer IN-.P, PAD2.P, T2A.E, T2B.E
- net LED: now also R7.1; no longer LED1.A, PAD1.P
- net N$4: now also C3.1, IC2.CE, IC2.VCC, LED2.A; no longer R5.2, T2A.B, T2B.B
- net N$5: now also R5.2; no longer T2A.C, T2B.C
- net SENSOR-: now also R3.1; no longer IN+.P, REG1A.VO, REG1B.VOUT
- net SOLAR: no longer R4.1
- net VCC: now also R4.1; no longer BAT+.P
Other:
- moved on the sheet: BAT+, BAT-, C2, IN+, R4, R5, REG1A, REG1B
