File: main.sch (EAGLE design)
At the start: 38 parts, among them IC1 ATTINY13A-SSH, IC2 TP4056-42-ESOP8, IC3 LM27313XMFX_NOPB, IC4 TPL5110DDCT, T1A 2N4401, T1B NPN, X1 MINI-USB-UX60A-MB-5ST, X2 332-02

Commit message: many updates
Parts:
- added R11: 10k, resistor:R-EU_R0805
- R1: value 510 -> 1k; device resistor:R-EU_M0805 -> resistor:R-EU_R0805
- R10, R2, R5, R6: device resistor:R-EU_M0805 -> resistor:R-EU_R0805
- R3: value 10k -> 1k; device resistor:R-EU_M0805 -> resistor:R-EU_R0805
- R7: value 510 -> 1k
- R9: device rcl:R-EU_R0603 -> rcl:R-EU_R0805
Connections:
- new net N$12: R11.2
- net RESET: now also R11.1
Changed lines of the file:
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@@
 <part name="PAD7" library="wirepad" library_urn="urn:adsk.eagle:library:412" deviceset="1,6/0,8" device="" package3d_urn="urn:adsk.eagle:package:30830/1"/>
 <part name="T1A" library="transistor" library_urn="urn:adsk.eagle:library:402" deviceset="*-NPN-" device="TO92" package3d_urn="urn:adsk.eagle:package:29893/2" value="2N4401"/>
-<part name="R2" library="resistor" library_urn="urn:adsk.eagle:library:348" deviceset="R-EU_" device="M0805" package3d_urn="urn:adsk.eagle:package:23556/1" value="10k"/>
+<part name="R2" library="resistor" library_urn="urn:adsk.eagle:library:348" deviceset="R-EU_" device="R0805" package3d_urn="urn:adsk.eagle:package:23553/2" value="10k"/>
 <part name="PUMP-" library="wirepad" library_urn="urn:adsk.eagle:library:412" deviceset="2,15/1,0" device="" package3d_urn="urn:adsk.eagle:package:30831/1"/>
 <part name="PUMP+" library="wirepad" library_urn="urn:adsk.eagle:library:412" deviceset="2,15/1,0" device="" package3d_urn="urn:adsk.eagle:package:30831/1"/>
@@
 <part name="PAD9" library="wirepad" library_urn="urn:adsk.eagle:library:412" deviceset="1,6/0,8" device="" package3d_urn="urn:adsk.eagle:package:30830/1"/>
 <part name="PAD10" library="wirepad" library_urn="urn:adsk.eagle:library:412" deviceset="1,6/0,8" device="" package3d_urn="urn:adsk.eagle:package:30830/1"/>
-<part name="R1" library="resistor" library_urn="urn:adsk.eagle:library:348" deviceset="R-EU_" device="M0805" package3d_urn="urn:adsk.eagle:package:23556/1" value="510"/>
+<part name="R1" library="resistor" library_urn="urn:adsk.eagle:library:348" deviceset="R-EU_" device="R0805" package3d_urn="urn:adsk.eagle:package:23553/2" value="1k"/>
 <part name="B-" library="wirepad" library_urn="urn:adsk.eagle:library:412" deviceset="1,6/0,8" device="" package3d_urn="urn:adsk.eagle:package:30830/1"/>
 <part name="GND3" library="supply1" library_urn="urn:adsk.eagle:library:371" deviceset="GND" device=""/>
@@
 <part name="GND5" library="supply1" library_urn="urn:adsk.eagle:library:371" deviceset="GND" device=""/>
 <part name="REG1A" library="linear" library_urn="urn:adsk.eagle:library:262" deviceset="78*" device="L" package3d_urn="urn:adsk.eagle:package:16416/2" technology="05"/>
-<part name="R6" library="resistor" library_urn="urn:adsk.eagle:library:348" deviceset="R-EU_" device="M0805" package3d_urn="urn:adsk.eagle:package:23556/1" value="10k"/>
+<part name="R6" library="resistor" library_urn="urn:adsk.eagle:library:348" deviceset="R-EU_" device="R0805" package3d_urn="urn:adsk.eagle:package:23553/2" value="10k"/>
 <part name="C1" library="rcl" library_urn="urn:adsk.eagle:library:334" deviceset="C-EU" device="C0805" package3d_urn="urn:adsk.eagle:package:23617/2" value="100nF"/>
 <part name="GND2" library="supply1" library_urn="urn:adsk.eagle:library:371" deviceset="GND" device=""/>
-<part name="R3" library="resistor" library_urn="urn:adsk.eagle:library:348" deviceset="R-EU_" device="M0805" package3d_urn="urn:adsk.eagle:package:23556/1" value="10k"/>
-<part name="R7" library="resistor" library_urn="urn:adsk.eagle:library:348" deviceset="R-EU_" device="M0805" package3d_urn="urn:adsk.eagle:package:23556/1" value="510"/>
+<part name="R3" library="resistor" library_urn="urn:adsk.eagle:library:348" deviceset="R-EU_" device="R0805" package3d_urn="urn:adsk.eagle:package:23553/2" value="1k"/>
+<part name="R7" library="resistor" library_urn="urn:adsk.eagle:library:348" deviceset="R-EU_" device="M0805" package3d_urn="urn:adsk.eagle:package:23556/1" value="1k"/>
 <part name="IC2" library="1EDI60I12AF" deviceset="TP4056-42-ESOP8" device=""/>
 <part name="C3" library="rcl" library_urn="urn:adsk.eagle:library:334" deviceset="C-EU" device="C3216" package3d_urn="urn:adsk.eagle:package:23628/2" value="10uF"/>
@@
 <part name="R8" library="rcl" library_urn="urn:adsk.eagle:library:334" deviceset="R-EU_" device="R0603" package3d_urn="urn:adsk.eagle:package:23555/3" value="10k"/>
 <part name="LED2" library="led" library_urn="urn:adsk.eagle:library:259" deviceset="LED" device="SML0805" package3d_urn="urn:adsk.eagle:package:15830/1"/>
-<part name="R9" library="rcl" library_urn="urn:adsk.eagle:library:334" deviceset="R-EU_" device="R0603" package3d_urn="urn:adsk.eagle:package:23555/3" value="1.2k"/>
+<part name="R9" library="rcl" library_urn="urn:adsk.eagle:library:334" deviceset="R-EU_" device="R0805" package3d_urn="urn:adsk.eagle:package:23553/2" value="1.2k"/>
 <part name="GND7" library="supply1" library_urn="urn:adsk.eagle:library:371" deviceset="GND" device=""/>
 <part name="X1" library="con-hirose" library_urn="urn:adsk.eagle:library:152" deviceset="MINI-USB-" device="UX60A-MB-5ST" package3d_urn="urn:adsk.eagle:package:7263/1"/>
@@
 <part name="IC3" library="1EDI60I12AF" deviceset="LM27313XMFX_NOPB" device=""/>
 <part name="GND1" library="supply1" library_urn="urn:adsk.eagle:library:371" deviceset="GND" device=""/>
-<part name="R5" library="resistor" library_urn="urn:adsk.eagle:library:348" deviceset="R-EU_" device="M0805" package3d_urn="urn:adsk.eagle:package:23556/1" value="10k"/>
+<part name="R5" library="resistor" library_urn="urn:adsk.eagle:library:348" deviceset="R-EU_" device="R0805" package3d_urn="urn:adsk.eagle:package:23553/2" value="10k"/>
 <part name="X2" library="con-garry" library_urn="urn:adsk.eagle:library:147" deviceset="332-02" device="" package3d_urn="urn:adsk.eagle:package:6810/1"/>
 <part name="GND10" library="supply1" library_urn="urn:adsk.eagle:library:371" deviceset="GND" device=""/>
 <part name="IC4" library="SamacSys" deviceset="TPL5110DDCT" device=""/>
 <part name="GND11" library="supply1" library_urn="urn:adsk.eagle:library:371" deviceset="GND" device=""/>
-<part name="R10" library="resistor" library_urn="urn:adsk.eagle:library:348" deviceset="R-EU_" device="M0805" package3d_urn="urn:adsk.eagle:package:23556/1" value="100k"/>
+<part name="R10" library="resistor" library_urn="urn:adsk.eagle:library:348" deviceset="R-EU_" device="R0805" package3d_urn="urn:adsk.eagle:package:23553/2" value="100k"/>
+<part name="R11" library="resistor" library_urn="urn:adsk.eagle:library:348" deviceset="R-EU_" device="R0805" package3d_urn="urn:adsk.eagle:package:23553/2" value="10k"/>
 </parts>
 <sheets>
@@
 <wire x1="137.16" y1="119.38" x2="88.9" y2="119.38" width="0.1524" layer="97"/>
 <text x="91.44" y="116.84" size="1.778" layer="97">Solar Charger</text>
-<wire x1="20.32" y1="60.96" x2="20.32" y2="15.24" width="0.1524" layer="97"/>
+<wire x1="20.32" y1="55.88" x2="20.32" y2="15.24" width="0.1524" layer="97"/>
 <wire x1="20.32" y1="15.24" x2="0" y2="15.24" width="0.1524" layer="97"/>
-<wire x1="0" y1="15.24" x2="0" y2="60.96" width="0.1524" layer="97"/>
-<wire x1="0" y1="60.96" x2="20.32" y2="60.96" width="0.1524" layer="97"/>
+<wire x1="0" y1="15.24" x2="0" y2="55.88" width="0.1524" layer="97"/>
+<wire x1="0" y1="55.88" x2="20.32" y2="55.88" width="0.1524" layer="97"/>
 <wire x1="48.26" y1="40.64" x2="86.36" y2="40.64" width="0.1524" layer="97"/>
 <wire x1="86.36" y1="40.64" x2="86.36" y2="15.24" width="0.1524" layer="97"/>
@@
 <wire x1="137.16" y1="17.78" x2="137.16" y2="48.26" width="0.1524" layer="97"/>
 <wire x1="137.16" y1="48.26" x2="106.68" y2="48.26" width="0.1524" layer="97"/>
-<text x="25.4" y="30.48" size="1.778" layer="97" rot="R90">Solar Voltage Sensor</text>
-<wire x1="35.56" y1="60.96" x2="35.56" y2="15.24" width="0.1524" layer="97"/>
+<text x="25.4" y="17.78" size="1.778" layer="97" rot="R90">Solar Voltage Sensor</text>
+<wire x1="35.56" y1="48.26" x2="35.56" y2="15.24" width="0.1524" layer="97"/>
 <wire x1="35.56" y1="15.24" x2="22.86" y2="15.24" width="0.1524" layer="97"/>
-<wire x1="35.56" y1="60.96" x2="22.86" y2="60.96" width="0.1524" layer="97"/>
-<wire x1="22.86" y1="60.96" x2="22.86" y2="15.24" width="0.1524" layer="97"/>
+<wire x1="35.56" y1="48.26" x2="22.86" y2="48.26" width="0.1524" layer="97"/>
+<wire x1="22.86" y1="48.26" x2="22.86" y2="15.24" width="0.1524" layer="97"/>
 <text x="50.8" y="83.82" size="1.778" layer="97" rot="R90">Low Power Sleep</text>
 <wire x1="48.26" y1="127" x2="48.26" y2="73.66" width="0.1524" layer="97"/>
@@
 <attribute name="NAME" x="-7.62" y="49.53" size="1.778" layer="95"/>
 </instance>
-<instance part="GND8" gate="1" x="-15.24" y="25.4" smashed="yes">
-<attribute name="VALUE" x="-17.78" y="22.86" size="1.778" layer="96"/>
+<instance part="GND8" gate="1" x="-15.24" y="20.32" smashed="yes">
+<attribute name="VALUE" x="-17.78" y="17.78" size="1.778" layer="96"/>
 </instance>
 <instance part="P+5" gate="VCC" x="-15.24" y="76.2" smashed="yes" rot="R180">
@@
 <attribute name="NAME" x="59.69" y="115.3414" size="1.778" layer="95" rot="R180"/>
 <attribute name="VALUE" x="59.69" y="120.142" size="1.778" layer="96" rot="R180"/>
+</instance>
+<instance part="R11" gate="G$1" x="10.16" y="58.42" smashed="yes" rot="R180">
+<attribute name="NAME" x="8.89" y="62.0014" size="1.778" layer="95" rot="R180"/>
+<attribute name="VALUE" x="13.97" y="61.722" size="1.778" layer="96" rot="R180"/>
 </instance>
 </instances>
@@
 <pinref part="GND8" gate="1" pin="GND"/>
 <pinref part="X1" gate="G$1" pin="5"/>
-<wire x1="-15.24" y1="27.94" x2="-15.24" y2="33.02" width="0.1524" layer="91"/>
+<wire x1="-15.24" y1="22.86" x2="-15.24" y2="33.02" width="0.1524" layer="91"/>
 </segment>
 <segment>
@@
 <label x="40.64" y="58.42" size="1.778" layer="95"/>
 <wire x1="38.1" y1="58.42" x2="50.8" y2="58.42" width="0.1524" layer="91"/>
+<pinref part="R11" gate="G$1" pin="1"/>
+<wire x1="15.24" y1="58.42" x2="38.1" y2="58.42" width="0.1524" layer="91"/>
+<junction x="38.1" y="58.42"/>
 </segment>
 </net>
@@
 </segment>
 </net>
+<net name="N$12" class="0">
+<segment>
+<pinref part="R11" gate="G$1" pin="2"/>
+<wire x1="5.08" y1="58.42" x2="-2.54" y2="58.42" width="0.1524" layer="91"/>
+</segment>
+</net>
+<net name="N$13" class="0">
+<segment>
+<wire x1="-2.54" y1="58.42" x2="-2.54" y2="45.72" width="0.1524" layer="91"/>
+<wire x1="-2.54" y1="45.72" x2="-7.62" y2="45.72" width="0.1524" layer="91"/>
+</segment>
+</net>

Commit message: updates
Parts:
- R11: device resistor:R-EU_R0805 -> resistor:R-EU_R0603
- R3: value 1k -> 330R
- R9: value 1.2k -> 2.2k
Connections:
- net UART_TX renamed SENSOR+
- removed net SENSOR/PUMP: IC1.PB0, PAD5.P, R1.2, X1.3
- removed net SOLAR: IC1.PB1, IC3.!SHDN, IC4.DONE, PAD6.P, REG1A.GND, X1.4
- new net NPN+: IC1.PB1, PAD6.P, R1.2, X1.4
- new net SOLAR_REG+/-: IC1.PB0, IC3.!SHDN, IC4.DONE, PAD5.P, REG1A.GND, X1.3
Other:
- moved on the sheet: PUMP-, R1, R2, T1A, T1B

Commit message: rev 0.8 (usbtiny built-in)
Parts:
- added D1, D2: BZX84CSMD, diode:BZX84CSMD
- added IC5: ATTINY13A-SSH, STM32F103RBT6:ATTINY13A-SSH
- added R12: 68R, resistor:R-EU_R0603
- added R13: 1.5k, resistor:R-EU_R0603
- added R14: 0R, resistor:R-EU_R0402
- C4: device rcl:C-EUC3216 -> rcl:C-EUC1206
- R11: value 10k -> 68R
- R7: device resistor:R-EU_M0805 -> resistor:R-EU_R0603
- R9: device rcl:R-EU_R0805 -> rcl:R-EU_R0603
Connections:
- new net N$10: IC5.PB4, R11.2
- new net N$13: D1.C, R11.1, R13.2, X1.2
- new net N$14: D2.C, R12.1, X1.3
- new net N$15: IC5.PB1, R14.1
- net GND: now also D1.A, D2.A, IC5.GND
- net LED: now also IC5.PB2; no longer X1.2
- net N$12: now also IC5.PB3, R12.2; no longer R11.2
- net N$5: now also IC5.VCC, R13.1
- net NPN+: now also R14.2; no longer X1.4
- net RESET: now also IC5.PB5; no longer R11.1
- net SOLAR_REG+/-: now also IC5.PB0; no longer X1.3
Other:
- note added: "ATTINY85"
- note added: "USBTINY Programmer"
- moved on the sheet: LED1, PUMP+, R11, R5, R6, R7, X1
