File: main.sch (EAGLE design)
At the start: 50 parts, among them IC1 ATTINY13A-SSH, IC2 TP4056-42-ESOP8, IC3 LM27313XMFX_NOPB, IC4 TPL5110DDCT, IC5 ATTINY13A-SSH, T1A 2N4401, T1B NPN, X1 MINI-USB-UX60A-MB-5ST

Commit message: firmware updates
Parts:
- JP1: device pinhead:PINHD-1X2/90 -> pinhead:PINHD-1X2
- renumbered REG1A to REG1
Changed lines of the file:
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@@
 <?xml version="1.0" encoding="utf-8"?>
 <!DOCTYPE eagle SYSTEM "eagle.dtd">
-<eagle version="9.6.0">
+<eagle version="9.6.1">
 <drawing>
 <settings>
@@
 <part name="C2" library="rcl" library_urn="urn:adsk.eagle:library:334" deviceset="CPOL-EU" device="E2.5-7" package3d_urn="urn:adsk.eagle:package:23345/1" value="1000uF"/>
 <part name="GND5" library="supply1" library_urn="urn:adsk.eagle:library:371" deviceset="GND" device=""/>
-<part name="REG1A" library="linear" library_urn="urn:adsk.eagle:library:262" deviceset="78*" device="L" package3d_urn="urn:adsk.eagle:package:16416/2" technology="05"/>
+<part name="REG1" library="linear" library_urn="urn:adsk.eagle:library:262" deviceset="78*" device="L" package3d_urn="urn:adsk.eagle:package:16416/2" technology="05"/>
 <part name="R6" library="resistor" library_urn="urn:adsk.eagle:library:348" deviceset="R-EU_" device="R0805" package3d_urn="urn:adsk.eagle:package:23553/2" value="10k"/>
 <part name="C1" library="rcl" library_urn="urn:adsk.eagle:library:334" deviceset="C-EU" device="C0805" package3d_urn="urn:adsk.eagle:package:23617/2" value="100nF"/>
@@
 <part name="R16" library="resistor" library_urn="urn:adsk.eagle:library:348" deviceset="R-EU_" device="R0603" package3d_urn="urn:adsk.eagle:package:23555/2" value="100R"/>
 <part name="R17" library="resistor" library_urn="urn:adsk.eagle:library:348" deviceset="R-EU_" device="R0603" package3d_urn="urn:adsk.eagle:package:23555/2" value="100R"/>
-<part name="JP1" library="pinhead" library_urn="urn:adsk.eagle:library:325" deviceset="PINHD-1X2" device="/90" package3d_urn="urn:adsk.eagle:package:22437/2"/>
+<part name="JP1" library="pinhead" library_urn="urn:adsk.eagle:library:325" deviceset="PINHD-1X2" device="" package3d_urn="urn:adsk.eagle:package:22435/2"/>
 <part name="GND6" library="supply1" library_urn="urn:adsk.eagle:library:371" deviceset="GND" device=""/>
 <part name="GND9" library="supply1" library_urn="urn:adsk.eagle:library:371" deviceset="GND" device=""/>
@@
 <attribute name="VALUE" x="33.02" y="86.36" size="1.778" layer="96"/>
 </instance>
-<instance part="REG1A" gate="A1" x="111.76" y="99.06" smashed="yes">
+<instance part="REG1" gate="A1" x="111.76" y="99.06" smashed="yes">
 <attribute name="VALUE" x="109.22" y="97.155" size="1.778" layer="96"/>
 </instance>
@@
 <wire x1="101.6" y1="88.9" x2="121.92" y2="88.9" width="0.1524" layer="91"/>
 <label x="106.68" y="86.36" size="1.778" layer="95"/>
-<pinref part="REG1A" gate="A1" pin="VI"/>
+<pinref part="REG1" gate="A1" pin="VI"/>
 <wire x1="101.6" y1="88.9" x2="101.6" y2="99.06" width="0.1524" layer="91"/>
 <junction x="101.6" y="88.9"/>
@@
 <wire x1="104.14" y1="76.2" x2="104.14" y2="81.28" width="0.1524" layer="91"/>
 <junction x="104.14" y="81.28"/>
-<pinref part="REG1A" gate="A1" pin="VO"/>
+<pinref part="REG1" gate="A1" pin="VO"/>
 <wire x1="121.92" y1="99.06" x2="132.08" y2="99.06" width="0.1524" layer="91"/>
 <wire x1="132.08" y1="99.06" x2="132.08" y2="81.28" width="0.1524" layer="91"/>
@@
 <net name="N$18" class="0">
 <segment>
-<pinref part="REG1A" gate="A1" pin="GND"/>
+<pinref part="REG1" gate="A1" pin="GND"/>
 <wire x1="111.76" y1="91.44" x2="91.44" y2="91.44" width="0.1524" layer="91"/>
 <pinref part="IC3" gate="G$1" pin="!SHDN"/>
