File: usbasp/hardware/usbasp.brd (EAGLE design)
At the start: 34.9 x 16.5 mm, 25 parts, among them IC1 ATMEGA8-16A, Q2 12Mhz, X1 USB-A-H

Commit message: many updates
Parts:
- moved C1 0.81 mm to (21.5, 3.17), flipped to the bottom
- moved VCCOUT 0.38 mm to (25.4, 8.64)
- moved D1 0.25 mm to (7.62, 11.8)
- moved D2 0.25 mm to (7.62, 4.70)
- flipped C3 to the bottom
- flipped Q2 to the top, turned to 0 degrees
Routing:
- net SELFPROG: track 18.0 -> 16.8 mm
- net RESET: track 22.2 -> 23.2 mm
- net XTAL1: track 14.3 -> 15.0 mm
- net VCC: track 83.6 -> 83.0 mm
- net XTAL2: track 5.33 -> 5.54 mm, vias 0 -> 1
- net GND: vias 9 -> 8

Commit message: added usbtiny + many updates
Parts:
- added R8: 10k, rcl:M0805
- added R9: 1k, rcl:M0805
- moved SELF 0.13 mm to (25.3, 3.17)
- moved SLOWSCK 0.13 mm to (25.3, 13.3)
- moved VCCOUT 0.13 mm to (25.3, 8.64)
Connections:
- new net N$1: ISP1.1, R9.1
- net GND: now also R8.1
- net MISO: now also R9.2; no longer ISP1.1
- net N$11: now also R8.2
Routing:
- net N$11: track 7.83 -> 16.8 mm
- net N$1: track 0.00 -> 4.31 mm
Changed lines of the file:
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@@
 <attribute name="VALUE" x="33.655" y="16.51" size="1.27" layer="27" rot="R180"/>
 </element>
-<element name="SLOWSCK" library="pinhead" package="1X02" value="" x="25.4" y="13.335" smashed="yes">
-<attribute name="NAME" x="22.7838" y="15.1638" size="1.27" layer="25" ratio="10"/>
-<attribute name="VALUE" x="22.86" y="10.16" size="1.27" layer="27"/>
+<element name="SLOWSCK" library="pinhead" package="1X02" value="" x="25.273" y="13.335" smashed="yes">
+<attribute name="NAME" x="22.6568" y="15.1638" size="1.27" layer="25" ratio="10"/>
+<attribute name="VALUE" x="22.733" y="10.16" size="1.27" layer="27"/>
 </element>
 <element name="R5" library="rcl" package="M0805" value="1k" x="32.385" y="2.54" smashed="yes" rot="MR180">
@@
 <attribute name="VALUE" x="31.115" y="16.51" size="1.27" layer="28" rot="MR180"/>
 </element>
-<element name="SELF" library="pinhead" package="1X02" value="" x="25.4" y="3.175" smashed="yes">
-<attribute name="NAME" x="22.7838" y="5.0038" size="1.27" layer="25" ratio="10"/>
-<attribute name="VALUE" x="22.86" y="0" size="1.27" layer="27"/>
+<element name="SELF" library="pinhead" package="1X02" value="" x="25.273" y="3.175" smashed="yes">
+<attribute name="NAME" x="22.6568" y="5.0038" size="1.27" layer="25" ratio="10"/>
+<attribute name="VALUE" x="22.733" y="0" size="1.27" layer="27"/>
 </element>
 <element name="IC1" library="avr" package="TQFP32-08" value="ATMEGA8-16A" x="16.51" y="9.525" smashed="yes">
@@
 <attribute name="VALUE" x="26.67" y="1.905" size="1.27" layer="28" rot="MR90"/>
 </element>
-<element name="VCCOUT" library="pinhead" package="1X02" value="" x="25.4" y="8.636" smashed="yes" rot="R180">
-<attribute name="NAME" x="28.0162" y="6.8072" size="1.27" layer="25" ratio="10" rot="R180"/>
-<attribute name="VALUE" x="27.94" y="11.811" size="1.27" layer="27" rot="R180"/>
+<element name="VCCOUT" library="pinhead" package="1X02" value="" x="25.273" y="8.636" smashed="yes" rot="R180">
+<attribute name="NAME" x="27.8892" y="6.8072" size="1.27" layer="25" ratio="10" rot="R180"/>
+<attribute name="VALUE" x="27.813" y="11.811" size="1.27" layer="27" rot="R180"/>
+</element>
+<element name="R8" library="rcl" package="M0805" value="10k" x="16.51" y="14.351" smashed="yes" rot="MR180">
+<attribute name="NAME" x="15.24" y="13.081" size="1.27" layer="26" rot="MR180"/>
+<attribute name="VALUE" x="15.24" y="16.891" size="1.27" layer="28" rot="MR180"/>
+</element>
+<element name="R9" library="rcl" package="M0805" value="1k" x="29.21" y="11.049" smashed="yes" rot="R270">
+<attribute name="NAME" x="30.48" y="12.319" size="1.27" layer="25" rot="R270"/>
+<attribute name="VALUE" x="26.67" y="12.319" size="1.27" layer="27" rot="R270"/>
 </element>
 </elements>
@@
 <vertex x="34.925" y="16.51"/>
 </polygon>
+<contactref element="R8" pad="1"/>
 </signal>
 <signal name="VCC" class="1">
@@
 <contactref element="ISP1" pad="2"/>
 <contactref element="VCCOUT" pad="1"/>
-<wire x1="26.67" y1="8.636" x2="27.7876" y2="9.7536" width="0.4064" layer="16"/>
-<wire x1="27.7876" y1="9.7536" x2="29.2086" y2="9.7536" width="0.4064" layer="16"/>
+<wire x1="26.543" y1="8.636" x2="27.6606" y2="9.7536" width="0.4064" layer="16"/>
+<wire x1="27.6606" y1="9.7536" x2="29.2086" y2="9.7536" width="0.4064" layer="16"/>
 <wire x1="29.2086" y1="9.7536" x2="29.21" y2="9.755" width="0.4064" layer="16"/>
 <wire x1="29.21" y1="9.755" x2="29.6686" y2="9.755" width="0.4064" layer="16"/>
@@
 <signal name="MISO">
 <contactref element="IC1" pad="16"/>
-<contactref element="ISP1" pad="1"/>
 <wire x1="19.31" y1="5.2324" x2="21.8948" y2="5.2324" width="0.2032" layer="1"/>
 <wire x1="21.8948" y1="5.2324" x2="22.1488" y2="5.4864" width="0.2032" layer="1"/>
@@
 <wire x1="30.5562" y1="9.017" x2="30.5562" y2="6.0198" width="0.2032" layer="16"/>
 <wire x1="30.5562" y1="9.017" x2="31.0896" y2="9.5504" width="0.2032" layer="16"/>
-<wire x1="31.0896" y1="9.5504" x2="31.7754" y2="9.5504" width="0.2032" layer="1"/>
-<wire x1="31.7754" y1="9.5504" x2="33.02" y2="10.795" width="0.2032" layer="1"/>
 <via x="30.6832" y="5.8928" extent="1-16" drill="0.508"/>
 <via x="31.0896" y="9.5504" extent="1-16" drill="0.508"/>
+<contactref element="R9" pad="2"/>
+<wire x1="31.0896" y1="9.5504" x2="30.541" y2="10.099" width="0.254" layer="1"/>
+<wire x1="30.541" y1="10.099" x2="29.21" y2="10.099" width="0.254" layer="1"/>
 </signal>
 <signal name="SCK">
@@
 <wire x1="20.32" y1="14.224" x2="21.1328" y2="14.224" width="0.254" layer="1"/>
 <wire x1="21.1328" y1="14.224" x2="21.5392" y2="13.8176" width="0.254" layer="1"/>
-<wire x1="21.5392" y1="13.8176" x2="23.6474" y2="13.8176" width="0.254" layer="1"/>
-<wire x1="23.6474" y1="13.8176" x2="24.13" y2="13.335" width="0.254" layer="1"/>
+<wire x1="21.5392" y1="13.8176" x2="23.5204" y2="13.8176" width="0.254" layer="1"/>
+<wire x1="23.5204" y1="13.8176" x2="24.003" y2="13.335" width="0.254" layer="1"/>
 </signal>
 <signal name="SELFPROG">
@@
 <wire x1="23.7744" y1="5.2832" x2="26.0096" y2="5.2832" width="0.254" layer="16"/>
 <wire x1="26.0096" y1="5.2832" x2="26.6192" y2="4.6736" width="0.254" layer="16"/>
-<wire x1="26.6192" y1="4.6736" x2="26.6192" y2="3.2258" width="0.254" layer="16"/>
-<wire x1="26.6192" y1="3.2258" x2="26.67" y2="3.175" width="0.254" layer="16"/>
+<wire x1="26.6192" y1="4.6736" x2="26.6192" y2="3.2512" width="0.254" layer="16"/>
+<wire x1="26.6192" y1="3.2512" x2="26.543" y2="3.175" width="0.254" layer="16"/>
 <via x="16.6624" y="11.9888" extent="1-16" drill="0.508"/>
 </signal>
@@
 <contactref element="SELF" pad="1"/>
 <contactref element="ISP1" pad="5"/>
-<wire x1="24.13" y1="1.9812" x2="24.13" y2="3.175" width="0.254" layer="16"/>
-<wire x1="23.0632" y1="0.9144" x2="24.13" y2="1.9812" width="0.254" layer="16"/>
+<wire x1="24.003" y1="1.8542" x2="24.003" y2="3.175" width="0.254" layer="16"/>
+<wire x1="23.0632" y1="0.9144" x2="24.003" y2="1.8542" width="0.254" layer="16"/>
 <wire x1="17.9832" y1="0.9144" x2="23.0632" y2="0.9144" width="0.254" layer="16"/>
 <wire x1="17.0688" y1="1.8288" x2="17.9832" y2="0.9144" width="0.254" layer="16"/>
@@
 <wire x1="17.71" y1="3.486" x2="17.71" y2="5.2324" width="0.254" layer="1"/>
 <wire x1="17.0688" y1="2.8448" x2="17.71" y2="3.486" width="0.254" layer="1"/>
-<wire x1="24.13" y1="3.175" x2="24.13" y2="4.0132" width="0.2032" layer="1"/>
-<wire x1="24.13" y1="4.0132" x2="25.1968" y2="5.08" width="0.2032" layer="1"/>
+<wire x1="24.003" y1="3.175" x2="24.003" y2="3.8862" width="0.2032" layer="1"/>
+<wire x1="24.003" y1="3.8862" x2="25.1968" y2="5.08" width="0.2032" layer="1"/>
 <wire x1="25.1968" y1="5.08" x2="31.2928" y2="5.08" width="0.2032" layer="1"/>
 <wire x1="31.2928" y1="5.08" x2="31.9278" y2="5.715" width="0.2032" layer="1"/>
@@
 <contactref element="R7" pad="2"/>
 <contactref element="VCCOUT" pad="2"/>
-<wire x1="24.13" y1="7.1374" x2="24.13" y2="8.636" width="0.4064" layer="16"/>
-<wire x1="24.7904" y1="6.477" x2="24.13" y2="7.1374" width="0.4064" layer="16"/>
+<wire x1="24.003" y1="7.2644" x2="24.003" y2="8.636" width="0.4064" layer="16"/>
+<wire x1="24.7904" y1="6.477" x2="24.003" y2="7.2644" width="0.4064" layer="16"/>
 <wire x1="24.7904" y1="6.477" x2="26.858" y2="6.477" width="0.4064" layer="16"/>
 <wire x1="26.858" y1="6.477" x2="29.21" y2="4.125" width="0.4064" layer="16"/>
+<contactref element="R8" pad="2"/>
+<wire x1="17.46" y1="14.351" x2="23.175" y2="8.636" width="0.4064" layer="16"/>
+<wire x1="23.175" y1="8.636" x2="24.003" y2="8.636" width="0.4064" layer="16"/>
 </signal>
 <signal name="N$9">
@@
 <wire x1="14.51" y1="14.954" x2="14.0208" y2="15.4432" width="0.254" layer="1"/>
 </signal>
+<signal name="N$1">
+<contactref element="R9" pad="1"/>
+<contactref element="ISP1" pad="1"/>
+<wire x1="29.21" y1="11.999" x2="31.816" y2="11.999" width="0.254" layer="1"/>
+<wire x1="31.816" y1="11.999" x2="33.02" y2="10.795" width="0.254" layer="1"/>
+</signal>
 </signals>

Commit message: lots of updates
Parts:
- removed R8: 10k, rcl:M0805
- removed R9: 1k, rcl:M0805
- added LED1, LED2: (no value), led:CHIP-LED0805
- R7: value 10 -> 10R
- moved C3 0.92 mm to (11.6, 3.30)
- moved C4 0.76 mm to (1.02, 8.13)
- moved C5 0.25 mm to (15.0, 9.53)
- moved C1 0.13 mm to (21.5, 3.30)
Connections:
- removed net N$1: ISP1.1, R9.1
- net GND: now also LED1.C, LED2.C; no longer R8.1
- net MISO: now also ISP1.1; no longer R9.2
- net N$11: no longer R8.2
- net N$6: now also LED1.A
- net N$7: now also LED2.A
Routing:
- net N$11: track 16.8 -> 7.88 mm
- net N$7: track 7.47 -> 15.8 mm
- net N$1: track 4.31 -> 0.00 mm
- net N$6: track 5.66 -> 9.58 mm
- net XTAL2: track 5.54 -> 7.58 mm, vias 1 -> 0
- net GND: track 4.49 -> 5.70 mm, vias 8 -> 5
- net MISO: track 17.7 -> 18.5 mm
